Commit message: update_obj

File: install/imu_force_description/share/imu_force_description/model/my-cylinder.xacro (robot description, xacro)
@@ -6,5 +6,5 @@
 			<visual>
 				<geometry>
-					<cylinder length="0.5" radius="0.1"/>
+					<cylinder length="0.06" radius="0.032"/>
 				</geometry>
 				<origin rpy="0 0 0" xyz="0 0 0"/>
@@ -12,8 +12,8 @@
 			<collision>
 				<geometry>
-					<cylinder length="0.5" radius="0.1"/>
+					<cylinder length="0.06" radius="0.032"/>
 				</geometry>
 			</collision>
-			<xacro:inertial_cylinder mass="1" length="0.5" radius="0.1">
+			<xacro:inertial_cylinder mass="0.05" length="0.06" radius="0.032">
         		<origin xyz="0 0 0" rpy="0 0 0"/>
     		</xacro:inertial_cylinder>
