Commit message: spawn_cylinder in gazebo

File: install/imu_force_description/share/imu_force_description/model/gazebo.xacro (robot description, xacro)
@@ -1,12 +1,8 @@
 <?xml version="1.0"?>
-<robot>
-	<gazebo>
-		<plugin name="gazebo_ros_control" filename="libgazebo_ros_control.so">
-			<robotNamespace>/cylinder </robotNamespace>
-		</plugin>
-	</gazebo>
-	<gazebo reference="base_link">
-		<mu1>0.2</mu1>
-		<mu2>0.2</mu2>
+<robot xmlns:xacro="http://www.ros.org/wiki/xacro" >
+    <xacro:include filename="inertial.xacro"/>
+	<gazebo reference="cylinder">
+		<mu1>0.0</mu1>
+		<mu2>0.0</mu2>
 		<material>Gazebo/Green</material>
 	</gazebo>

File: install/imu_force_description/share/imu_force_description/model/my-cylinder.xacro (robot description, xacro)
@@ -2,5 +2,5 @@
 <robot xmlns:xacro="http://www.ros.org/wiki/xacro" name="my_cylinder">
 	<!-- Include the Gazebo definitions  -->
-	<!-- <xacro:include filename="gazebo.xacro"/> -->
+	<xacro:include filename="gazebo.xacro"/>
 		<link name="cylinder">
 			<visual>
@@ -8,18 +8,14 @@
 					<cylinder length="0.5" radius="0.1"/>
 				</geometry>
-				<!-- <origin rpy="0 0 0" xyz="0 0 0"/>					 -->
+				<origin rpy="0 0 0" xyz="0 0 0"/>
 			</visual>
-			<!-- <collision>
+			<collision>
 				<geometry>
-					<cylinder length="${base_link_length}"
-					radius="${base_link_radius}"/>
+					<cylinder length="0.5" radius="0.1"/>
 				</geometry>
-				<origin rpy="0 0 0" xyz="0 0 0"/>
 			</collision>
-			<inertial>
-				<origin rpy="0 0 0" xyz="0 0 0"/>
-				<mass value="1"/>
-				<inertia ixx="100" ixy="0" ixz="0" iyy="100" iyz="0" izz="100" />
-			</inertial> -->
+			<xacro:inertial_cylinder mass="1" length="0.5" radius="0.1">
+        		<origin xyz="0 0 0" rpy="0 0 0"/>
+    		</xacro:inertial_cylinder>
 		</link>
 </robot>

File: src/imu_force_description/model/gazebo.xacro (robot description, xacro)
@@ -1,21 +1,8 @@
 <?xml version="1.0"?>
-<robot>
-	<xacro:macro name="inertial_cylinder" params="mass length radius *origin">
-        <inertial>
-            <xacro:insert_block name="origin"/>
-            <mass value="${mass}" />
-            <inertia ixx="${(1/12) * mass * (3*radius*radius + length*length)}" ixy="0.0" ixz="0.0"
-                    iyy="${(1/12) * mass * (3*radius*radius + length*length)}" iyz="0.0"
-                    izz="${(1/2) * mass * (radius*radius)}" />
-        </inertial>
-    </xacro:macro>
-	<gazebo>
-		<plugin name="gazebo_ros_control" filename="libgazebo_ros_control.so">
-			<robotNamespace>/cylinder </robotNamespace>
-		</plugin>
-	</gazebo>
+<robot xmlns:xacro="http://www.ros.org/wiki/xacro" >
+    <xacro:include filename="inertial.xacro"/>
 	<gazebo reference="cylinder">
-		<mu1>0.2</mu1>
-		<mu2>0.2</mu2>
+		<mu1>0.0</mu1>
+		<mu2>0.0</mu2>
 		<material>Gazebo/Green</material>
 	</gazebo>

Commit message: add_ground truth position broad cast in rviz

File: install/imu_force_description/share/imu_force_description/model/gazebo.xacro (robot description, xacro)
@@ -2,4 +2,11 @@
 <robot xmlns:xacro="http://www.ros.org/wiki/xacro" >
     <xacro:include filename="inertial.xacro"/>
+	<gazebo>
+		<plugin name="ground_truth_plugin" filename="libgazebo_ros_p3d.so">
+			<update_rate>50.0</update_rate>
+			<body_name>cylinder</body_name>
+			<frame_name>world</frame_name>
+		</plugin>
+	</gazebo>
 	<gazebo reference="cylinder">
 		<mu1>0.0</mu1>

File: install/imu_force_description/share/imu_force_description/model/my-cylinder.xacro (robot description, xacro)
@@ -3,19 +3,19 @@
 	<!-- Include the Gazebo definitions  -->
 	<xacro:include filename="gazebo.xacro"/>
-		<link name="cylinder">
-			<visual>
-				<geometry>
-					<cylinder length="0.06" radius="0.032"/>
-				</geometry>
-				<origin rpy="0 0 0" xyz="0 0 0"/>
-			</visual>
-			<collision>
-				<geometry>
-					<cylinder length="0.06" radius="0.032"/>
-				</geometry>
-			</collision>
-			<xacro:inertial_cylinder mass="0.05" length="0.06" radius="0.032">
-        		<origin xyz="0 0 0" rpy="0 0 0"/>
-    		</xacro:inertial_cylinder>
-		</link>
+	<link name="cylinder">
+		<visual>
+			<geometry>
+				<cylinder length="0.06" radius="0.032"/>
+			</geometry>
+			<origin rpy="0 0 0" xyz="0 0 0"/>
+		</visual>
+		<collision>
+			<geometry>
+				<cylinder length="0.06" radius="0.032"/>
+			</geometry>
+		</collision>
+		<xacro:inertial_cylinder mass="0.05" length="0.06" radius="0.032">
+			<origin xyz="0 0 0" rpy="0 0 0"/>
+		</xacro:inertial_cylinder>
+	</link>
 </robot>
